Commit message: tune params

File: src/g1_description/urdf/g1_29_inspire.urdf (robot description, URDF)
Before this commit: robot g1_29dof_rev_1_0_with_inspire_hand_DFQ, 63 links, 62 joints
Links:
- added link tag_frame
Joints:
- added joint imu_in_torso_to_tag_frame: type fixed, parent imu_in_torso, child tag_frame, origin xyz=0.05 0 0 rpy=-1.5707963267948966 0 1.5707963267948966

Commit message: improve apriltag localization

File: src/g1_description/urdf/g1_29_inspire.urdf (robot description, URDF)
Before this commit: robot g1_29dof_rev_1_0_with_inspire_hand_DFQ, 64 links, 63 joints
Links:
- removed link tag_frame
- added link tag_mount_frame
Joints:
- removed joint imu_in_torso_to_tag_frame
- added joint imu_in_torso_to_tag_mount_frame: type fixed, parent imu_in_torso, child tag_mount_frame, origin xyz=0.05 0 0 rpy=-1.5707963267948966 0 -1.5707963267948966

Commit message: add extra configurations

File: src/g1_description/urdf/g1_29_inspire.urdf (robot description, URDF)
Before this commit: robot g1_29dof_rev_1_0_with_inspire_hand_DFQ, 64 links, 63 joints
Joints:
- joint L_index_intermediate_joint: axis 0 0 -1 -> (none); limit lower=0 upper=1.7 effort=1 velocity=0.5 -> (none); mimic joint=L_index_proximal_joint multiplier=1 offset=0 -> (none); type revolute -> fixed
- joint L_index_proximal_joint: axis 0 0 -1 -> (none); limit lower=0 upper=1.7 effort=1 velocity=0.5 -> (none); type revolute -> fixed
- joint L_middle_intermediate_joint: axis 0 0 -1 -> (none); limit lower=0 upper=1.7 effort=1 velocity=0.5 -> (none); mimic joint=L_middle_proximal_joint multiplier=1 offset=0 -> (none); type revolute -> fixed
- joint L_middle_proximal_joint: axis 0 0 -1 -> (none); limit lower=0 upper=1.7 effort=1 velocity=0.5 -> (none); type revolute -> fixed
- joint L_pinky_intermediate_joint: axis 0 0 -1 -> (none); limit lower=0 upper=1.7 effort=1 velocity=0.5 -> (none); mimic joint=L_pinky_proximal_joint multiplier=1 offset=0 -> (none); type revolute -> fixed
- joint L_pinky_proximal_joint: axis 0 0 -1 -> (none); limit lower=0 upper=1.7 effort=1 velocity=0.5 -> (none); type revolute -> fixed
- joint L_ring_intermediate_joint: axis 0 0 -1 -> (none); limit lower=0 upper=1.7 effort=1 velocity=0.5 -> (none); mimic joint=L_ring_proximal_joint multiplier=1 offset=0 -> (none); type revolute -> fixed
- joint L_ring_proximal_joint: axis 0 0 -1 -> (none); limit lower=0 upper=1.7 effort=1 velocity=0.5 -> (none); type revolute -> fixed
- joint L_thumb_distal_joint: axis 0 0 -1 -> (none); limit lower=0 upper=1.2 effort=1 velocity=0.5 -> (none); mimic joint=L_thumb_proximal_pitch_joint multiplier=2.4 offset=0 -> (none); type revolute -> fixed
- joint L_thumb_intermediate_joint: axis 0 0 -1 -> (none); limit lower=0 upper=0.8 effort=1 velocity=0.5 -> (none); mimic joint=L_thumb_proximal_pitch_joint multiplier=1.6 offset=0 -> (none); type revolute -> fixed
- joint L_thumb_proximal_pitch_joint: axis 0 0 -1 -> (none); limit lower=-0.1 upper=0.6 effort=1 velocity=0.5 -> (none); type revolute -> fixed
- joint L_thumb_proximal_yaw_joint: axis 0 0 1 -> (none); limit lower=-0.1 upper=1.3 effort=1 velocity=0.5 -> (none); type revolute -> fixed
- joint R_index_intermediate_joint: axis 0 0 1 -> (none); limit lower=0 upper=1.7 effort=1 velocity=0.5 -> (none); mimic joint=R_index_proximal_joint multiplier=1 offset=0 -> (none); type revolute -> fixed
- joint R_index_proximal_joint: axis 0 0 1 -> (none); limit lower=0 upper=1.7 effort=1 velocity=0.5 -> (none); type revolute -> fixed
- joint R_middle_intermediate_joint: axis 0 0 1 -> (none); limit lower=0 upper=1.7 effort=1 velocity=0.5 -> (none); mimic joint=R_middle_proximal_joint multiplier=1 offset=0 -> (none); type revolute -> fixed
- joint R_middle_proximal_joint: axis 0 0 1 -> (none); limit lower=0 upper=1.7 effort=1 velocity=0.5 -> (none); type revolute -> fixed
- joint R_pinky_intermediate_joint: axis 0 0 1 -> (none); limit lower=0 upper=1.7 effort=1 velocity=0.5 -> (none); mimic joint=R_pinky_proximal_joint multiplier=1 offset=0 -> (none); type revolute -> fixed
- joint R_pinky_proximal_joint: axis 0 0 1 -> (none); limit lower=0 upper=1.7 effort=1 velocity=0.5 -> (none); type revolute -> fixed
- joint R_ring_intermediate_joint: axis 0 0 1 -> (none); limit lower=0 upper=1.7 effort=1 velocity=0.5 -> (none); mimic joint=R_ring_proximal_joint multiplier=1 offset=0 -> (none); type revolute -> fixed
- joint R_ring_proximal_joint: axis 0 0 1 -> (none); limit lower=0 upper=1.7 effort=1 velocity=0.5 -> (none); type revolute -> fixed
- joint R_thumb_distal_joint: axis 0 0 1 -> (none); limit lower=0 upper=1.2 effort=1 velocity=0.5 -> (none); mimic joint=R_thumb_proximal_pitch_joint multiplier=2.4 offset=0 -> (none); type revolute -> fixed
- joint R_thumb_intermediate_joint: axis 0 0 1 -> (none); limit lower=0 upper=0.8 effort=1 velocity=0.5 -> (none); mimic joint=R_thumb_proximal_pitch_joint multiplier=1.6 offset=0 -> (none); type revolute -> fixed
- joint R_thumb_proximal_pitch_joint: axis 0 0 1 -> (none); limit lower=-0.1 upper=0.6 effort=1 velocity=0.5 -> (none); type revolute -> fixed
- joint R_thumb_proximal_yaw_joint: axis 0 0 -1 -> (none); limit lower=-0.1 upper=1.3 effort=1 velocity=0.5 -> (none); type revolute -> fixed
